Commit message: add gitignore

File: install/simulation/share/simulation/urdf/first_robot.urdf.xacro (robot description, xacro)
@@ -1,41 +1 @@
-<?xml version="1.0"?>
-<robot xmlns:xacro="http://www.ros.org/wiki/xacro" name="first_robot">
-    <!-- 声明 base 模块 -->
-    <xacro:macro name="base_link" params="length radius">
-        <link name="base_link">
-            <visual>
-                <origin xyz="0 0 0" rpy="0 0 0" />
-                <geometry>
-                    <cylinder length="${length}" radius="${length}" />
-                </geometry>
-                <material name="blue">
-                    <color rgba="0.1 0.1 1.0 0.5" />
-                </material>
-            </visual>
-        </link>
-    </xacro:macro>
-    <!-- 声明 IMU 模块 -->
-    <xacro:macro name="imu_link" params="imu_name xyz">
-        <link name="${imu_name}_link">
-            <visual>
-                <origin xyz="0 0 0" rpy="0 0 0" />
-                <geometry>
-                    <box size="0.02 0.02 0.02" />
-                </geometry>
-            </visual>
-            <material name="black">
-                <color rgba="0 0 0 0.5" />
-            </material>
-        </link>
-        <joint name="${imu_name}_joint" type="fixed">
-            <parent link="base_link" />
-            <child link="${imu_name}_link" />
-            <origin xyz="${xyz}" />
-        </joint>
-    </xacro:macro>
-    <!-- 传递参数调用 base_link 模块 -->
-    <xacro:base_link length="0.12" radius="0.1" />
-    <!-- 传递参数调用 imu 模块 -->
-    <xacro:imu_link imu_name="imu_up" xyz="0 0 0.02" />
-    <xacro:imu_link imu_name="imu_down" xyz="0 0 -0.02" />
-</robot>
+/home/rm/2025-sentry-navi/src/simulation/urdf/first_robot.urdf.xacro

File: install/simulation/share/simulation/urdf/fishbot/actuator/caster.urdf.xacro (robot description, xacro)
@@ -1,39 +1 @@
-<?xml version="1.0"?>
-<robot xmlns:xacro="http://www.ros.org/wiki/xacro">
-   <xacro:include filename="$(find simulation)/urdf/fishbot/common_inertia.xacro" />
-    <xacro:macro name="caster_xacro" params="caster_name xyz">
-        <link name="${caster_name}_caster_link">
-            <visual>
-                <origin xyz="0 0 0" rpy="0 0 0" />
-                <geometry>
-                    <sphere radius="0.016" />
-                </geometry>
-                <material name="black">
-                    <color rgba="0.0 0.0 0.0 0.8"/>
-                </material>
-            </visual>
-            <collision>
-                <origin xyz="0 0 0" rpy="0 0 0" />
-                <geometry>
-                    <sphere radius="0.016" />
-                </geometry>
-                <material name="black">
-                    <color rgba="0.0 0.0 0.0 0.8"/>
-                </material>
-            </collision>
-            <xacro:sphere_inertia m="0.01" r="0.016" />
-        </link>
-        <gazebo reference="${caster_name}_caster_link">
-            <mu1 value="0.0" />
-            <mu2 value="0.0" />
-            <kp value="1000000000.0" />
-            <kd value="1.0" />
-        </gazebo>
-        <joint name="${caster_name}_caster_joint" type="fixed">
-            <parent link="base_link" />
-            <child link="${caster_name}_caster_link" />
-            <origin xyz="${xyz}" />
-            <axis xyz="0 0 0" />
-        </joint>
-    </xacro:macro>
-</robot>
+/home/rm/2025-sentry-navi/src/simulation/urdf/fishbot/actuator/caster.urdf.xacro

File: install/simulation/share/simulation/urdf/fishbot/actuator/wheel.urdf.xacro (robot description, xacro)
@@ -1,39 +1 @@
-<?xml version="1.0"?>
-<robot xmlns:xacro="http://www.ros.org/wiki/xacro">
-   <xacro:include filename="$(find simulation)/urdf/fishbot/common_inertia.xacro" />
-    <xacro:macro name="wheel_xacro" params="wheel_name xyz">
-        <link name="${wheel_name}_wheel_link">
-            <visual>
-                <origin xyz="0 0 0" rpy="1.57079 0 0" />
-                <geometry>
-                    <cylinder length="0.04" radius="0.032" />
-                </geometry>
-                <material name="black">
-                    <color rgba="0.0 0.0 0.0 0.8"/>
-                </material>
-            </visual>
-            <collision>
-                <origin xyz="0 0 0" rpy="1.57079 0 0" />
-                <geometry>
-                    <cylinder length="0.04" radius="0.032" />
-                </geometry>
-                <material name="black">
-                    <color rgba="0.0 0.0 0.0 0.8"/>
-                </material>
-            </collision>
-            <xacro:cylinder_inertia m="0.1" h="0.04" r="0.032"/>
-        </link>
-        <gazebo reference="${wheel_name}_wheel_link">
-            <mu1 value="20.0" />
-            <mu2 value="20.0" />
-            <kp value="1000000000.0" />
-            <kd value="1.0" />
-        </gazebo>
-        <joint name="${wheel_name}_wheel_joint" type="continuous">
-            <parent link="base_link" />
-            <child link="${wheel_name}_wheel_link" />
-            <origin xyz="${xyz}" />
-            <axis xyz="0 1 0" />
-        </joint>
-    </xacro:macro>
-</robot>
+/home/rm/2025-sentry-navi/src/simulation/urdf/fishbot/actuator/wheel.urdf.xacro

File: install/simulation/share/simulation/urdf/fishbot/base.urdf.xacro (robot description, xacro)
@@ -1,33 +1 @@
-<?xml version="1.0"?>
-<robot xmlns:xacro="http://www.ros.org/wiki/xacro">
-   <xacro:include filename="$(find simulation)/urdf/fishbot/common_inertia.xacro" />
-    <xacro:macro name="base_xacro" params="length radius">
-     <link name="base_footprint" />
-        <joint name="base_joint" type="fixed">
-            <parent link="base_footprint" />
-            <child link="base_link" />
-            <origin xyz="0.0 0.0 ${length/2.0+0.032-0.001}" rpy="0 0 0" />
-        </joint>
-        <link name="base_link">
-            <visual>
-                <origin xyz="0 0 0.0" rpy="0 0 0" />
-                <geometry>
-                    <cylinder length="${length}" radius="${length}" />
-                </geometry>
-                <material name="blue">
-                    <color rgba="0.1 0.1 1.0 0.5"/>
-                </material>
-            </visual>
-            <collision>
-                <origin xyz="0 0 0.0" rpy="0 0 0" />
-                <geometry>
-                    <cylinder length="${length}" radius="${length}" />
-                </geometry>
-                <material name="blue">
-                    <color rgba="0.1 0.1 1.0 0.5"/>
-                </material>
-            </collision>
-            <xacro:cylinder_inertia m="1.0" r="${radius}" h="${length}"/>
-        </link>
-    </xacro:macro>
-</robot>
+/home/rm/2025-sentry-navi/src/simulation/urdf/fishbot/base.urdf.xacro

File: install/simulation/share/simulation/urdf/fishbot/common_inertia.xacro (robot description, xacro)
@@ -1,21 +1 @@
-<?xml version="1.0"?>
-<robot xmlns:xacro="http://ros.org/wiki/xacro">
-    <xacro:macro name="box_inertia" params="m w h d">
-        <inertial>
-            <mass value="${m}" />
-            <inertia ixx="${(m/12) * (h*h + d*d)}" ixy="0.0" ixz="0.0" iyy="${(m/12) * (w*w + d*d)}" iyz="0.0" izz="${(m/12) * (w*w + h*h)}" />
-        </inertial>
-    </xacro:macro>
-    <xacro:macro name="cylinder_inertia" params="m r h">
-        <inertial>
-            <mass value="${m}" />
-            <inertia ixx="${(m/12) * (3*r*r + h*h)}" ixy="0" ixz="0" iyy="${(m/12) * (3*r*r + h*h)}" iyz="0" izz="${(m/2) * (r*r)}" />
-        </inertial>
-    </xacro:macro>
-    <xacro:macro name="sphere_inertia" params="m r">
-        <inertial>
-            <mass value="${m}" />
-            <inertia ixx="${(2/5) * m * (r*r)}" ixy="0.0" ixz="0.0" iyy="${(2/5) * m * (r*r)}" iyz="0.0" izz="${(2/5) * m * (r*r)}" />
-        </inertial>
-    </xacro:macro>
-</robot>
+/home/rm/2025-sentry-navi/src/simulation/urdf/fishbot/common_inertia.xacro

File: install/simulation/share/simulation/urdf/fishbot/fishbot.ros2_control.xacro (robot description, xacro)
@@ -1,45 +1 @@
-<?xml version="1.0"?>
-<robot xmlns:xacro="http://www.ros.org/wiki/xacro">
-    <xacro:macro name="fishbot_ros2_control">
-    <ros2_control name="FishBotGazeboSystem" type="system">
-            <hardware>
-                <plugin>gazebo_ros2_control/GazeboSystem</plugin>
-            </hardware>
-            <joint name="left_wheel_joint">
-                <command_interface name="velocity">
-                    <param name="min">-5</param>
-                    <param name="max">5</param>
-                </command_interface>
-                <command_interface name="effort">
-                    <param name="min">-0.5</param>
-                    <param name="max">0.5</param>
-                </command_interface>
-                <state_interface name="position" />
-                <state_interface name="velocity" />
-                <state_interface name="effort" />
-            </joint>
-            <joint name="right_wheel_joint">
-                <command_interface name="velocity">
-                    <param name="min">-5</param>
-                    <param name="max">5</param>
-                </command_interface>
-                <command_interface name="effort">
-                    <param name="min">-0.5</param>
-                    <param name="max">0.5</param>
-                </command_interface>
-                <state_interface name="position" />
-                <state_interface name="velocity" />
-                <state_interface name="effort" />
-            </joint>
-        </ros2_control>
-        <gazebo>
-        <plugin filename="libgazebo_ros2_control.so" name="gazebo_ros2_control">
-            <parameters>$(find simulation)/config/fishbot_ros2_controller.yaml</parameters>
-            <ros>
-                <remapping>/fishbot_diff_drive_controller/cmd_vel_unstamped:=/cmd_vel</remapping>
-                <remapping>/fishbot_diff_drive_controller/odom:=/odom</remapping>
-            </ros>
-        </plugin>
-</gazebo>
-    </xacro:macro>
-</robot>
+/home/rm/2025-sentry-navi/src/simulation/urdf/fishbot/fishbot.ros2_control.xacro

File: install/simulation/share/simulation/urdf/fishbot/fishbot.urdf.xacro (robot description, xacro)
@@ -1,28 +1 @@
-<?xml version="1.0"?>
-<robot xmlns:xacro="http://www.ros.org/wiki/xacro" name="fishbot">
-    <xacro:include filename="$(find simulation)/urdf/fishbot/base.urdf.xacro" />
-    <!-- 传感器组件 -->
-    <xacro:include filename="$(find simulation)/urdf/fishbot/sensor/imu.urdf.xacro" />
-    <xacro:include filename="$(find simulation)/urdf/fishbot/sensor/laser.urdf.xacro" />
-    <xacro:include filename="$(find simulation)/urdf/fishbot/sensor/camera.urdf.xacro" />
-     <!-- 执行器组件 -->
-    <xacro:include filename="$(find simulation)/urdf/fishbot/actuator/wheel.urdf.xacro" />
-    <xacro:include filename="$(find simulation)/urdf/fishbot/actuator/caster.urdf.xacro" />
-    <xacro:base_xacro length="0.12" radius="0.1" />
-    <!-- 传感器 -->
-    <xacro:imu_xacro xyz="0 0 0.02" />
-    <xacro:laser_xacro xyz="0 0 0.10" />
-    <xacro:camera_xacro xyz="0.10 0 0.075" />
-    <!-- 执行器主动轮+从动轮 -->
-    <xacro:wheel_xacro wheel_name="left" xyz="0 0.10 -0.06" />
-    <xacro:wheel_xacro wheel_name="right" xyz="0 -0.10 -0.06" />
-    <xacro:caster_xacro caster_name="front" xyz="0.08 0.0 -0.076" />
-    <xacro:caster_xacro caster_name="back" xyz="-0.08 0.0 -0.076" />
-    <!-- Gazebo 插件 -->
-    <xacro:include filename="$(find simulation)/urdf/fishbot/plugins/gazebo_control_plugin.xacro" />
-    <!-- <xacro:gazebo_control_plugin /> -->
-    <xacro:include filename="$(find simulation)/urdf/fishbot/fishbot.ros2_control.xacro" />
-    <xacro:fishbot_ros2_control />
-    <xacro:include filename="$(find simulation)/urdf/fishbot/plugins/gazebo_sensor_plugin.xacro" />
-    <xacro:gazebo_sensor_plugin />
-</robot>
+/home/rm/2025-sentry-navi/src/simulation/urdf/fishbot/fishbot.urdf.xacro

File: install/simulation/share/simulation/urdf/fishbot/plugins/gazebo_control_plugin.xacro (robot description, xacro)
@@ -1,30 +1 @@
-<?xml version="1.0"?>
-<robot xmlns:xacro="http://www.ros.org/wiki/xacro">
-    <xacro:macro name="gazebo_control_plugin">
-        <gazebo>
-            <plugin name='diff_drive' filename='libgazebo_ros_diff_drive.so'>
-                <ros>
-                    <namespace>/</namespace>
-                    <remapping>cmd_vel:=cmd_vel</remapping>
-                    <remapping>odom:=odom</remapping>
-                </ros>
-                <update_rate>30</update_rate>
-                <!-- wheels -->
-                <left_joint>left_wheel_joint</left_joint>
-                <right_joint>right_wheel_joint</right_joint>
-                <!-- kinematics -->
-                <wheel_separation>0.2</wheel_separation>
-                <wheel_diameter>0.064</wheel_diameter>
-                <!-- limits -->
-                <max_wheel_torque>20</max_wheel_torque>
-                <max_wheel_acceleration>1.0</max_wheel_acceleration>
-                <!-- output -->
-                <publish_odom>true</publish_odom>
-                <publish_odom_tf>true</publish_odom_tf>
-                <publish_wheel_tf>true</publish_wheel_tf>
-                <odometry_frame>odom</odometry_frame>
-                <robot_base_frame>base_footprint</robot_base_frame>
-            </plugin>
-        </gazebo>
-   </xacro:macro>
-</robot>
+/home/rm/2025-sentry-navi/src/simulation/urdf/fishbot/plugins/gazebo_control_plugin.xacro

File: install/simulation/share/simulation/urdf/fishbot/plugins/gazebo_sensor_plugin.xacro (robot description, xacro)
@@ -1,138 +1 @@
-<?xml version="1.0"?>
-<robot xmlns:xacro="http://www.ros.org/wiki/xacro">
-    <xacro:macro name="gazebo_sensor_plugin">
-        <gazebo reference="laser_link">
-            <sensor name="laserscan" type="ray">
-                <plugin name="laserscan" filename="libgazebo_ros_ray_sensor.so">
-                    <ros>
-                        <namespace>/</namespace>
-                        <remapping>~/out:=scan</remapping>
-                    </ros>
-                    <output_type>sensor_msgs/LaserScan</output_type>
-                    <frame_name>laser_link</frame_name>
-                </plugin>
-                <always_on>true</always_on>
-                <visualize>false</visualize>
-                <update_rate>10</update_rate>
-                <pose>0 0 0 0 0 0</pose>
-								<!-- 激光传感器配置 -->
-                <ray>
-                    <!-- 设置扫描范围 -->
-                    <scan>
-                        <horizontal>
-                            <samples>360</samples>
-                            <resolution>1.000000</resolution>
-                            <min_angle>0.000000</min_angle>
-                            <max_angle>6.280000</max_angle>
-                        </horizontal>
-                    </scan>
-                    <!-- 设置扫描距离 -->
-                    <range>
-                        <min>0.120000</min>
-                        <max>8.0</max>
-                        <resolution>0.015000</resolution>
-                    </range>
-                    <!-- 设置噪声 -->
-                    <noise>
-                        <type>gaussian</type>
-                        <mean>0.0</mean>
-                        <stddev>0.01</stddev>
-                    </noise>
-                </ray>
-            </sensor>
-        </gazebo>
-<gazebo reference="imu_link">
-    <sensor name="imu_sensor" type="imu">
-        <plugin name="imu_plugin" filename="libgazebo_ros_imu_sensor.so">
-            <ros>
-                <namespace>/</namespace>
-                <remapping>~/out:=imu</remapping>
-            </ros>
-            <initial_orientation_as_reference>false</initial_orientation_as_reference>
-        </plugin>
-        <update_rate>100</update_rate>
-        <always_on>true</always_on>
-        <!-- 六轴噪声设置 -->
-        <imu>
-            <angular_velocity>
-                <x>
-                    <noise type="gaussian">
-                        <mean>0.0</mean>
-                        <stddev>2e-4</stddev>
-                        <bias_mean>0.0000075</bias_mean>
-                        <bias_stddev>0.0000008</bias_stddev>
-                    </noise>
-                </x>
-                <y>
-                    <noise type="gaussian">
-                        <mean>0.0</mean>
-                        <stddev>2e-4</stddev>
-                        <bias_mean>0.0000075</bias_mean>
-                        <bias_stddev>0.0000008</bias_stddev>
-                    </noise>
-                </y>
-                <z>
-                    <noise type="gaussian">
-                        <mean>0.0</mean>
-                        <stddev>2e-4</stddev>
-                        <bias_mean>0.0000075</bias_mean>
-                        <bias_stddev>0.0000008</bias_stddev>
-                    </noise>
-                </z>
-            </angular_velocity>
-            <linear_acceleration>
-                <x>
-                    <noise type="gaussian">
-                        <mean>0.0</mean>
-                        <stddev>1.7e-2</stddev>
-                        <bias_mean>0.1</bias_mean>
-                        <bias_stddev>0.001</bias_stddev>
-                    </noise>
-                </x>
-                <y>
-                    <noise type="gaussian">
-                        <mean>0.0</mean>
-                        <stddev>1.7e-2</stddev>
-                        <bias_mean>0.1</bias_mean>
-                        <bias_stddev>0.001</bias_stddev>
-                    </noise>
-                </y>
-                <z>
-                    <noise type="gaussian">
-                        <mean>0.0</mean>
-                        <stddev>1.7e-2</stddev>
-                        <bias_mean>0.1</bias_mean>
-                        <bias_stddev>0.001</bias_stddev>
-                    </noise>
-                </z>
-            </linear_acceleration>
-        </imu>
-    </sensor>
-</gazebo>
-    </xacro:macro>
-<gazebo reference="camera_link">
-    <sensor type="depth" name="camera_sensor">
-        <plugin name="depth_camera" filename="libgazebo_ros_camera.so">
-            <frame_name>camera_optical_link</frame_name>
-        </plugin>
-        <always_on>true</always_on>
-        <update_rate>10</update_rate>
-        <camera name="camera">
-            <horizontal_fov>1.5009831567</horizontal_fov>
-            <image>
-                <width>800</width>
-                <height>600</height>
-                <format>R8G8B8</format>
-            </image>
-            <distortion>
-                <k1>0.0</k1>
-                <k2>0.0</k2>
-                <k3>0.0</k3>
-                <p1>0.0</p1>
-                <p2>0.0</p2>
-                <center>0.5 0.5</center>
-            </distortion>
-        </camera>
-    </sensor>
-</gazebo>
-</robot>
+/home/rm/2025-sentry-navi/src/simulation/urdf/fishbot/plugins/gazebo_sensor_plugin.xacro

File: install/simulation/share/simulation/urdf/fishbot/sensor/camera.urdf.xacro (robot description, xacro)
@@ -1,39 +1 @@
-<?xml version="1.0"?>
-<robot xmlns:xacro="http://www.ros.org/wiki/xacro">
-   <xacro:include filename="$(find simulation)/urdf/fishbot/common_inertia.xacro" />
-    <xacro:macro name="camera_xacro" params="xyz">
-        <!-- ============相机模块================ -->
-        <link name="camera_link">
-            <visual>
-                <origin xyz="0 0 0.0" rpy="0 0 0" />
-                <geometry>
-                    <box size="0.02 0.10 0.02" />
-                </geometry>
-                <material name="black">
-                    <color rgba="0.0 0.0 0.0 0.8"/>
-                </material>
-            </visual>
-            <collision>
-                <origin xyz="0 0 0.0" rpy="0 0 0" />
-                <geometry>
-                    <box size="0.02 0.10 0.02" />
-                </geometry>
-                <material name="black">
-                    <color rgba="0.0 0.0 0.0 0.8"/>
-                </material>
-            </collision>
-            <xacro:box_inertia m="0.01" w="0.02" h="0.10" d="0.02" />
-        </link>
-        <link name="camera_optical_link"></link>
-        <joint name="camera_optical_joint" type="fixed">
-            <parent link="camera_link" />
-            <child link="camera_optical_link" />
-            <origin xyz="0 0 0" rpy="${-pi/2} 0 ${-pi/2}" />
-        </joint>
-        <joint name="camera_joint" type="fixed">
-            <parent link="base_link" />
-            <child link="camera_link" />
-            <origin xyz="${xyz}" />
-        </joint>
-    </xacro:macro>
-</robot>
+/home/rm/2025-sentry-navi/src/simulation/urdf/fishbot/sensor/camera.urdf.xacro

File: install/simulation/share/simulation/urdf/fishbot/sensor/imu.urdf.xacro (robot description, xacro)
@@ -1,32 +1 @@
-<?xml version="1.0"?>
-<robot xmlns:xacro="http://www.ros.org/wiki/xacro">
-   <xacro:include filename="$(find simulation)/urdf/fishbot/common_inertia.xacro" />
-    <xacro:macro name="imu_xacro" params="xyz">
-        <link name="imu_link">
-            <visual>
-                <origin xyz="0 0 00" rpy="0 0 0" />
-                <geometry>
-                    <box size="0.02 0.02 0.02" />
-                </geometry>
-                <material name="black">
-                    <color rgba="0 0 0 0.8" />
-                </material>
-            </visual>
-            <collision>
-                <origin xyz="0 0 00" rpy="0 0 0" />
-                <geometry>
-                    <box size="0.02 0.02 0.02" />
-                </geometry>
-                <material name="black">
-                    <color rgba="0 0 0 0.8" />
-                </material>
-            </collision>
-            <xacro:box_inertia m="0.01" w="0.02" d="0.02" h="0.02"/>
-        </link>
-        <joint name="imu_joint" type="fixed">
-            <parent link="base_link" />
-            <child link="imu_link" />
-            <origin xyz="${xyz}" />
-        </joint>
-    </xacro:macro>
-</robot>
+/home/rm/2025-sentry-navi/src/simulation/urdf/fishbot/sensor/imu.urdf.xacro
